File: pcb/watch/watch.kicad_pcb (KiCad board)
At the start: 2 copper layers, 61.5 x 31.6 mm, 428 parts

Commit message: fuck fuck fuck I made it too small
Parts:
- removed R100, R101, R102, R103, R104, R105, R106, R107 (x6), R108, R109, R110, R111, R112, R113, R114, R115, R116, R117, R118, R119, R120, R121, R122, R123, R124, R125, R126, R127, R128, R129, R130, R131, R132, R133, R134, R135, R136, R137, R138, R139, R140, R141, R142, R143, R144, R145, R146, R147, R148, R149, R150, R151, R152, R153, R154, R155, R156, R157, R158, R159, R160, R161, R162, R163, R164, R165, R166, R167, R168, R169, R170, R171, R172, R173, R174, R175, R176, R177, R178, R179, R180, R181, R182, R183, R184, R185, R186, R187, R188, R189, R190, R191, R192, R193, R194, R195, R196, R197, R198, R199, R200, R201, R202, R203, R204, R205, R206, R207, R208, R209, R210, R211, R212, R213, R214, R215, R216, R217, R218, R219, R220, R221, R222, R223, R224, R225, R226, R227, R228, R229, R230, R231, R232, R233, R234, R235, R236, R237, R238, R239, R240, R241, R242, R243, R244, R245, R246, R247, R248, R249, R250, R251, R252, R253, R254, R255, R256, R257, R258, R259, R260, R261, R262, R263, R264, R265, R266, R267, R268, R269, R270, R271, R272, R273, R274, R275, R276, R312, R313, R314, R315, R316, R317, R318, R319, R320, R321, R322, R323, R324, R325, R326, R327, R328, R329, R330, R331, R332, R333, R334, R335, R336, R337, R338, R339, R340, R341 (x2), R342, R343, R344, R345, R346, R347, R348, R349, R350, R351, R352, R353, R354, R355, R356, R357, R358, R359, R360, R361, R362, R363, R364, R365, R366, R367, R368, R369, R370, R371, R372, R373, R374, R375, R376, R377, R378, R379, R380, R381, R382, R383, R384, R385, R386, R387, R388, R389, R390, R391, R392, R393, R394, R395, R396, R397, R398, R399, R400, R401, R402, R403, R404, R405, R406, R407, R408, R409, R410, R411, R412, R413, R414, R415, R416, R417, R418, R419, R420, R421, R422, R423, R424, R425, R426, R427, R428, R429, R430, R431, R432, R433, R434, R435, R436, R437, R438, R439, R440, R441, R442, R443, R444, R445, R446, R447, R448, R449, R450, R451, R452, R453, R59, R62, R63, R64, R65, R66, R67, R68, R69, R70, R71, R72, R73, R74, R75, R76, R77, R78, R79, R80, R81, R82, R83, R84, R85, R86, R87, R88, R89, R90, R91, R92, R93, R94, R95, R96, R97, R98, R99: 87, Resistor_SMD:R_0402_1005Metric
- removed the R2 at (67.2, 135.6)
- removed the R2 at (86.7, 142.1)
- removed the R2 at (86.7, 144.0)
- removed the R2 at (90.0, 140.6)
- removed the R2 at (86.7, 139.0)
- removed the R2 at (75.6, 135.6)
- removed the R2 at (78.5, 142.2)
- removed the R2 at (70.4, 137.1)
- removed the R2 at (80.3, 142.1)
- removed the R2 at (65.7, 137.1)
- removed the R2 at (73.4, 145.6)
- removed the R2 at (88.2, 135.6)
- removed the R2 at (85.0, 142.1)
- removed the R2 at (85.0, 139.0)
- removed the R2 at (90.2, 135.6)
- removed the R2 at (224.1, 153.8)
- removed the R2 at (65.7, 144.0)
- removed the R2 at (80.3, 139.0)
- removed the R2 at (72.1, 137.1)
- removed the R2 at (69.2, 135.6)
- removed the R2 at (75.4, 140.6)
- removed the R2 at (72.1, 142.1)
- removed the R2 at (72.1, 144.0)
- removed the R2 at (69.0, 140.6)
- removed the R2 at (91.4, 142.1)
- removed the R2 at (91.4, 137.1)
- removed the R2 at (70.4, 142.1)
- removed the R2 at (88.0, 140.6)
- removed the R2 at (86.7, 137.1)
- removed the R2 at (76.9, 137.1)
- removed the R2 at (73.4, 140.6)
- removed the R2 at (81.6, 140.6)
- removed the R2 at (67.0, 145.6)
- removed the R2 at (80.3, 144.0)
- removed the R2 at (76.9, 139.0)
- removed the R2 at (76.9, 144.0)
- removed the R2 at (69.0, 145.6)
- removed the R2 at (85.0, 137.1)
- removed the R2 at (72.1, 139.0)
- removed the R2 at (76.9, 142.1)
- removed the R2 at (78.5, 138.8)
- removed the R2 at (81.8, 135.6)
- removed the R2 at (70.4, 144.0)
- removed the R2 at (81.6, 145.6)
- removed the R2 at (83.7, 135.6)
- removed the R2 at (90.0, 145.6)
- removed the R2 at (73.6, 135.6)
- removed the R2 at (88.0, 145.6)
- removed the R2 at (224.1, 155.5)
- removed the R2 at (80.3, 137.1)
- removed the R2 at (91.4, 144.0)
- removed the R2 at (65.7, 139.0)
- removed the R2 at (75.4, 145.6)
- removed the R2 at (91.4, 139.0)
- removed the R2 at (83.5, 145.6)
- removed the R2 at (258.3, 153.0)
- removed the R2 at (65.7, 142.1)
- removed the R2 at (83.5, 140.6)
- removed the R2 at (85.0, 144.0)
- removed the R2 at (67.0, 140.6)
- removed the R2 at (70.4, 139.0)
- removed REF** (x3): ST_WLCSP-81_Die463, Package_CSP:ST_WLCSP-81_Die463
- added D1: LED_Small_Filled, footprints:LED_0402_1005Metric, F.Cu at (0.00, -12.0)
- added D10: LED_Small_Filled, LED_SMD:LED_0402_1005Metric, F.Cu at (-10.9, -5.11)
- added D11: LED_Small_Filled, footprints:LED_0402_1005Metric, F.Cu at (-11.4, -3.71)
- added D12: LED_Small_Filled, LED_SMD:LED_0402_1005Metric, F.Cu at (-11.8, -2.25)
- added D13: LED_Small_Filled, LED_SMD:LED_0402_1005Metric, F.Cu at (-12.0, -0.75)
- added D14: LED_Small_Filled, LED_SMD:LED_0402_1005Metric, F.Cu at (-12.0, 0.75)
- added D15: LED_Small_Filled, LED_SMD:LED_0402_1005Metric, F.Cu at (-11.8, 2.25)
- added D16: LED_Small_Filled, LED_SMD:LED_0402_1005Metric, F.Cu at (-11.4, 3.71)
- added D17: LED_Small_Filled, LED_SMD:LED_0402_1005Metric, F.Cu at (-10.9, 5.11)
- added D18: LED_Small_Filled, LED_SMD:LED_0402_1005Metric, F.Cu at (-10.1, 6.43)
- added D19: LED_Small_Filled, LED_SMD:LED_0402_1005Metric, F.Cu at (-9.25, 7.65)
- added D2: LED_Small_Filled, LED_SMD:LED_0402_1005Metric, F.Cu at (-1.50, -11.9)
- added D20: LED_Small_Filled, LED_SMD:LED_0402_1005Metric, F.Cu at (-8.21, 8.75)
- added D21: LED_Small_Filled, footprints:LED_0402_1005Metric, F.Cu at (-7.05, 9.71)
- added D22: LED_Small_Filled, LED_SMD:LED_0402_1005Metric, F.Cu at (-5.78, 10.5)
- added D23: LED_Small_Filled, LED_SMD:LED_0402_1005Metric, F.Cu at (-4.42, 11.2)
- added D24: LED_Small_Filled, LED_SMD:LED_0402_1005Metric, F.Cu at (-2.98, 11.6)
- added D25: LED_Small_Filled, LED_SMD:LED_0402_1005Metric, F.Cu at (-1.50, 11.9)
- added D26: LED_Small_Filled, LED_SMD:LED_0402_1005Metric, F.Cu at (0.00, 12.0)
- added D27: LED_Small_Filled, LED_SMD:LED_0402_1005Metric, F.Cu at (1.50, 11.9)
- added D28: LED_Small_Filled, LED_SMD:LED_0402_1005Metric, F.Cu at (2.98, 11.6)
- added D29: LED_Small_Filled, LED_SMD:LED_0402_1005Metric, F.Cu at (4.42, 11.2)
- added D3: LED_Small_Filled, LED_SMD:LED_0402_1005Metric, F.Cu at (-2.98, -11.6)
- added D30: LED_Small_Filled, LED_SMD:LED_0402_1005Metric, F.Cu at (5.78, 10.5)
- added D31: LED_Small_Filled, footprints:LED_0402_1005Metric, F.Cu at (7.05, 9.71)
- added D32: LED_Small_Filled, LED_SMD:LED_0402_1005Metric, F.Cu at (8.21, 8.75)
- added D33: LED_Small_Filled, LED_SMD:LED_0402_1005Metric, F.Cu at (9.25, 7.65)
- added D34: LED_Small_Filled, LED_SMD:LED_0402_1005Metric, F.Cu at (10.1, 6.43)
- added D35: LED_Small_Filled, LED_SMD:LED_0402_1005Metric, F.Cu at (10.9, 5.11)
- added D36: LED_Small_Filled, LED_SMD:LED_0402_1005Metric, F.Cu at (11.4, 3.71)
- added D37: LED_Small_Filled, LED_SMD:LED_0402_1005Metric, F.Cu at (11.8, 2.25)
- added D38: LED_Small_Filled, LED_SMD:LED_0402_1005Metric, F.Cu at (12.0, 0.75)
- added D39: LED_Small_Filled, LED_SMD:LED_0402_1005Metric, F.Cu at (12.0, -0.75)
- added D4: LED_Small_Filled, LED_SMD:LED_0402_1005Metric, F.Cu at (-4.42, -11.2)
- added D40: LED_Small_Filled, LED_SMD:LED_0402_1005Metric, F.Cu at (11.8, -2.25)
- added D41: LED_Small_Filled, footprints:LED_0402_1005Metric, F.Cu at (11.4, -3.71)
- added D42: LED_Small_Filled, LED_SMD:LED_0402_1005Metric, F.Cu at (10.9, -5.11)
- added D43: LED_Small_Filled, LED_SMD:LED_0402_1005Metric, F.Cu at (10.1, -6.43)
- added D44: LED_Small_Filled, LED_SMD:LED_0402_1005Metric, F.Cu at (9.25, -7.65)
- added D45: LED_Small_Filled, LED_SMD:LED_0402_1005Metric, F.Cu at (8.21, -8.75)
- added D46: LED_Small_Filled, LED_SMD:LED_0402_1005Metric, F.Cu at (7.05, -9.71)
- added D47: LED_Small_Filled, LED_SMD:LED_0402_1005Metric, F.Cu at (5.78, -10.5)
- added D48: LED_Small_Filled, LED_SMD:LED_0402_1005Metric, F.Cu at (4.42, -11.2)
- added D49: LED_Small_Filled, LED_SMD:LED_0402_1005Metric, F.Cu at (2.98, -11.6)
- added D5: LED_Small_Filled, LED_SMD:LED_0402_1005Metric, F.Cu at (-5.78, -10.5)
- added D50: LED_Small_Filled, LED_SMD:LED_0402_1005Metric, F.Cu at (1.50, -11.9)
- added D51: LED_Small_Filled, LED_SMD:LED_0402_1005Metric, F.Cu at (0.00, -10.0)
- added D52: LED_Small_Filled, LED_SMD:LED_0402_1005Metric, F.Cu at (-2.59, -9.66)
- added D53: LED_Small_Filled, LED_SMD:LED_0402_1005Metric, F.Cu at (-5.00, -8.66)
- added D54: LED_Small_Filled, LED_SMD:LED_0402_1005Metric, F.Cu at (-7.07, -7.07)
- added D55: LED_Small_Filled, LED_SMD:LED_0402_1005Metric, F.Cu at (-8.66, -5.00)
- added D56: LED_Small_Filled, LED_SMD:LED_0402_1005Metric, F.Cu at (-9.66, -2.59)
- added D57: LED_Small_Filled, LED_SMD:LED_0402_1005Metric, F.Cu at (-10.0, 0.00)
- added D58: LED_Small_Filled, LED_SMD:LED_0402_1005Metric, F.Cu at (-9.66, 2.59)
- added D59: LED_Small_Filled, LED_SMD:LED_0402_1005Metric, F.Cu at (-8.66, 5.00)
- added D6: LED_Small_Filled, LED_SMD:LED_0402_1005Metric, F.Cu at (-7.05, -9.71)
- added D60: LED_Small_Filled, LED_SMD:LED_0402_1005Metric, F.Cu at (-7.07, 7.07)
- added D61: LED_Small_Filled, LED_SMD:LED_0402_1005Metric, F.Cu at (-5.00, 8.66)
- added D62: LED_Small_Filled, LED_SMD:LED_0402_1005Metric, F.Cu at (-2.59, 9.66)
- added D63: LED_Small_Filled, LED_SMD:LED_0402_1005Metric, F.Cu at (0.00, 10.0)
- added D64: LED_Small_Filled, LED_SMD:LED_0402_1005Metric, F.Cu at (2.59, 9.66)
- added D65: LED_Small_Filled, LED_SMD:LED_0402_1005Metric, F.Cu at (5.00, 8.66)
- added D66: LED_Small_Filled, LED_SMD:LED_0402_1005Metric, F.Cu at (7.07, 7.07)
- added D67: LED_Small_Filled, LED_SMD:LED_0402_1005Metric, F.Cu at (8.66, 5.00)
- added D68: LED_Small_Filled, LED_SMD:LED_0402_1005Metric, F.Cu at (9.66, 2.59)
- added D69: LED_Small_Filled, LED_SMD:LED_0402_1005Metric, F.Cu at (10.0, 0.00)
- added D7: LED_Small_Filled, LED_SMD:LED_0402_1005Metric, F.Cu at (-8.21, -8.75)
- added D70: LED_Small_Filled, LED_SMD:LED_0402_1005Metric, F.Cu at (9.66, -2.59)
- added D71: LED_Small_Filled, LED_SMD:LED_0402_1005Metric, F.Cu at (8.66, -5.00)
- added D72: LED_Small_Filled, LED_SMD:LED_0402_1005Metric, F.Cu at (7.07, -7.07)
- added D73: LED_Small_Filled, LED_SMD:LED_0402_1005Metric, F.Cu at (5.00, -8.66)
- added D74: LED_Small_Filled, LED_SMD:LED_0402_1005Metric, F.Cu at (2.59, -9.66)
- added D8: LED_Small_Filled, LED_SMD:LED_0402_1005Metric, F.Cu at (-9.25, -7.65)
- added D9: LED_Small_Filled, LED_SMD:LED_0402_1005Metric, F.Cu at (-10.1, -6.43)
- added R1: R_Small_US, Resistor_SMD:R_0402_1005Metric, F.Cu at (0.00, -8.50)
- added R2: R_Small_US, Resistor_SMD:R_0402_1005Metric, F.Cu at (-8.08, -2.63)
- added R3: R_Small_US, Resistor_SMD:R_0402_1005Metric, F.Cu at (-5.00, 6.88)
- added R4: R_Small_US, Resistor_SMD:R_0402_1005Metric, F.Cu at (5.00, 6.88)
- added R5: R_Small_US, Resistor_SMD:R_0402_1005Metric, F.Cu at (8.08, -2.63)
- added R6: R_Small_US, Resistor_SMD:R_0402_1005Metric, F.Cu at (2.60, -6.00)
- added R7: R_Small_US, Resistor_SMD:R_0402_1005Metric, F.Cu at (2.60, -7.00)
- added R8: R_Small_US, Resistor_SMD:R_0402_1005Metric, F.Cu at (2.60, -8.00)
- added U1: STM32G031K8Ux, Package_DFN_QFN:UFQFPN-32-1EP_5x5mm_P0.5mm_EP3.5x3.5mm, F.Cu at (0.00, 0.00)
Routing:
- net /LED1: track 0.00 -> 89.1 mm, vias 0 -> 5
- net /LED5: track 0.00 -> 86.8 mm, vias 0 -> 5
- net /LED4: track 0.00 -> 84.7 mm, vias 0 -> 5
- net /LED2: track 0.00 -> 82.8 mm, vias 0 -> 5
- net /LED3: track 0.00 -> 82.7 mm, vias 0 -> 5
- net Net-(D51-K): track 0.00 -> 62.7 mm, vias 0 -> 5
- net Net-(D53-K): track 0.00 -> 61.8 mm, vias 0 -> 4
- net Net-(D55-K): track 0.00 -> 58.4 mm, vias 0 -> 4
- net /LED17: track 0.00 -> 30.7 mm
- net Net-(D11-A): track 0.00 -> 29.6 mm
- net Net-(D1-A): track 0.00 -> 29.2 mm
- net Net-(D31-A): track 0.00 -> 29.0 mm
- net Net-(D21-A): track 0.00 -> 28.7 mm
- net Net-(D41-A): track 0.00 -> 27.8 mm
- net /LED15: track 0.00 -> 27.2 mm, vias 0 -> 2
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Other:
- board size 61.5 x 31.6 mm -> 28 x 34.6 mm
- copper layers 2 -> 4
- board text removed: "12"
- board text removed: "24"
- board text removed: "30"
- board text removed: "60 90 deg leds"
- board text removed: "digital"

Commit message: eee
Parts:
- added BT1: LIR2032, footprints:LIR2032, B.Cu at (0.00, 0.00)
- added C1: 1u, footprints:C_0402_nosilk, F.Cu at (-2.32, 1.63)
- added C2: 1u, footprints:C_0402_nosilk, F.Cu at (-2.32, 4.49)
- added R10: 169k, footprints:LED_0402_nosilk, F.Cu at (-2.32, -0.36)
- added R9: 169k, footprints:LED_0402_nosilk, F.Cu at (-2.32, 0.64)
- added TP1: TestPoint_2Pole, footprints:tesptoint_tiny, F.Cu at (-9.20, 12.3)
- added TP2: TestPoint_2Pole, footprints:tesptoint_tiny, F.Cu at (8.50, 12.3)
- added TP3: TestPoint_2Pole, footprints:tesptoint_tiny, F.Cu at (-9.44, -12.5)
- added TP4: TestPoint_2Pole, footprints:tesptoint_tiny, F.Cu at (9.29, -12.5)
- added U2: TLV74130PDQNR, footprints:Texas_X2SON_nosilk, F.Cu at (-2.32, 3.06)
- D52, D53, D54, D55, D56, D57, D58, D59, D60, D61, D62, D63, D64, D65, D66, D67, D68, D69, D70, D71, D72, D73, D74: footprint LED_SMD:LED_0402_1005Metric -> footprints:LED_0402_nosilk
- R1, R2, R3, R4, R5, R6, R7, R8: footprint Resistor_SMD:R_0402_1005Metric -> footprints:R_0402_nosilk
- U1: footprint Package_DFN_QFN:UFQFPN-32-1EP_5x5mm_P0.5mm_EP3.5x3.5mm -> footprints:UFQFPN-32-nosilk
- moved U1 5.22 mm to (-2.80, -4.40)
Connections:
- U1 pad 1: /LED1 -> /LED15
- U1 pad 11: unconnected-(U1-PA4-Pad11) -> /LED10
- U1 pad 15: /LED10 -> unconnected-(U1-PB0-Pad15)
- U1 pad 2: /LED8 -> /LED3
- U1 pad 20: /LED5 -> /LED6
- U1 pad 21: /LED6 -> /LED5
- U1 pad 22: /LED14 -> unconnected-(U1-PA11/PA9-Pad22)
- U1 pad 23: unconnected-(U1-PA12/PA10-Pad23) -> /LED14
- U1 pad 24: unconnected-(U1-PA13-Pad24) -> /SWDIO
- U1 pad 25: /LED7 -> /SWCLK
- U1 pad 27: unconnected-(U1-PB3-Pad27) -> /LED7
- U1 pad 3: /LED15 -> GND
- U1 pad 31: unconnected-(U1-PB7-Pad31) -> /LED1
- U1 pad 32: unconnected-(U1-PB8-Pad32) -> /LED8
- U1 pad 33: Net-(U1-VSS-Pad33) -> GND
- U1 pad 4: unconnected-(U1-VDD-Pad4) -> VDD
- U1 pad 5: Net-(U1-VSS-Pad33) -> GND
- U1 pad 6: /LED3 -> unconnected-(U1-PF2-Pad6)
- U1 pad 7: unconnected-(U1-PA0-Pad7) -> Net-(U1-PA0)
Routing:
- net /coil_{+}: track 0.00 -> 652.3 mm, vias 0 -> 2
- net GND: track 0.00 -> 63.2 mm, vias 0 -> 1
- net VDD: track 0.00 -> 50.9 mm, vias 0 -> 2
- net +BATT: track 0.00 -> 33.5 mm, vias 0 -> 2
- net /LED3: track 82.7 -> 100.3 mm, vias 5 -> 6
- net /LED9: track 5.25 -> 19.8 mm
- net Net-(D21-A): track 28.7 -> 39.7 mm, vias 0 -> 2
- net /SWCLK: track 0.00 -> 10.4 mm, vias 0 -> 1
- net /LED4: track 84.7 -> 94.0 mm
- net /LED10: track 9.91 -> 18.5 mm
- net /LED8: track 5.45 -> 13.1 mm
- net /SWDIO: track 0.00 -> 7.28 mm, vias 0 -> 1
- net /LED15: track 27.2 -> 34.1 mm
- net /LED16: track 24.2 -> 29.3 mm
- net /LED14: track 24.7 -> 20.9 mm
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- added copper zone on F.Cu, net +BATT
- added copper zone on F.Cu, net GND
- added copper zone on F.Cu, net VDD
Other:
- outline, holes or cut-outs redrawn

Commit message: eeeee
Parts:
- moved C2 9.96 mm to (6.02, -0.95), turned to 180 degrees
- moved R10 9.36 mm to (6.02, 3.90), turned to 0 degrees
- moved U1 9.33 mm to (0.00, 4.50)
- moved U2 8.73 mm to (6.02, 0.48), turned to -90 degrees
- moved R9 8.64 mm to (6.02, 2.90), turned to 180 degrees
- moved C1 8.34 mm to (6.02, 1.91), turned to 180 degrees
Connections:
- U1 pad 1: /LED15 -> /LED8
- U1 pad 16: /LED11 -> unconnected-(U1-PB1-Pad16)
- U1 pad 17: /LED12 -> unconnected-(U1-PB2-Pad17)
- U1 pad 18: /LED13 -> unconnected-(U1-PA8-Pad18)
- U1 pad 19: /LED17 -> unconnected-(U1-PA9/NC-Pad19)
- U1 pad 2: /LED3 -> /LED15
- U1 pad 20: /LED6 -> unconnected-(U1-PC6-Pad20)
- U1 pad 21: /LED5 -> /LED17
- U1 pad 22: unconnected-(U1-PA11/PA9-Pad22) -> /LED11
- U1 pad 23: /LED14 -> /LED12
- U1 pad 26: /LED2 -> /LED14
- U1 pad 27: /LED7 -> /LED13
- U1 pad 28: unconnected-(U1-PB4-Pad28) -> /LED7
- U1 pad 29: unconnected-(U1-PB5-Pad29) -> /LED2
- U1 pad 3: GND -> /LED3
- U1 pad 30: unconnected-(U1-PB6-Pad30) -> /LED6
- U1 pad 31: /LED1 -> /LED5
- U1 pad 32: /LED8 -> /LED1
Routing:
- net /LED6: track 3.50 -> 33.0 mm, vias 0 -> 2
- net /LED13: track 4.30 -> 28.4 mm, vias 0 -> 2
- net /LED10: track 18.5 -> 34.7 mm
- net /LED4: track 94.0 -> 109.8 mm
- net /LED16: track 29.3 -> 44.8 mm
- net /SWDIO: track 7.28 -> 20.7 mm
- net /LED9: track 19.8 -> 33.2 mm
- net /LED3: track 100.3 -> 88.0 mm
- net /LED15: track 34.1 -> 23.2 mm
- net /LED8: track 13.1 -> 3.14 mm
- net /LED5: track 86.4 -> 95.9 mm, vias 5 -> 6
- net /SWCLK: track 10.4 -> 19.6 mm
- net /LED14: track 20.9 -> 30.0 mm
- net /LED12: track 3.21 -> 12.0 mm
- net /LED1: track 91.5 -> 82.9 mm
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
Commit message: better outline
Parts:
- moved R6 2.24 mm to (4.80, -6.40)
- moved R7 1.17 mm to (3.70, -7.40)
- moved R8 0.40 mm to (2.60, -8.40)
Routing:
- net GND: track 64.6 -> 23.7 mm
- net +BATT: track 36.8 -> 23.7 mm, vias 2 -> 3
- net /LED12: track 12.0 -> 19.6 mm
- net /LED11: track 10.9 -> 18.1 mm
- net Net-(D51-K): track 65.3 -> 63.3 mm
- net /LED17: track 35.5 -> 37.2 mm
- net /SWDIO: track 20.7 -> 21.9 mm
- net Net-(D53-K): track 65.1 -> 64.1 mm
- net /SWCLK: track 19.6 -> 18.7 mm
- net /LED16: track 44.8 -> 44.1 mm
- net /LED10: track 34.7 -> 34.0 mm
- net /LED4: track 109.8 -> 109.0 mm
- net /LED6: track 33.0 -> 32.5 mm
- net /LED9: track 33.2 -> 32.6 mm
- added copper zone on B.Cu, net +BATT
- added copper zone on In2.Cu, net +BATT
- added copper zone on B.Cu, net GND
Other:
- board size 28 x 34.6 mm -> 28 x 34.7 mm

Commit message: rev1 lol
Parts:
- removed TP1: TestPoint_2Pole, footprints:tesptoint_tiny
- added R11: 0, Resistor_SMD:R_0402_1005Metric, F.Cu at (-6.75, -5.75)
- added R12: 0, Resistor_SMD:R_0402_1005Metric, F.Cu at (-5.00, -7.00)
- added R13: 0, Resistor_SMD:R_0402_1005Metric, F.Cu at (5.49, 13.0)
- moved R8 1.35 mm to (1.70, -7.40)
Connections:
- TP2 pad 2: +BATT -> Net-(R13-Pad2)
- U1 pad 12: unconnected-(U1-PA5-Pad12) -> /LED17
- U1 pad 13: unconnected-(U1-PA6-Pad13) -> /LED11
- U1 pad 14: unconnected-(U1-PA7-Pad14) -> /LED12
- U1 pad 21: /LED17 -> unconnected-(U1-PA10/NC-Pad21)
- U1 pad 22: /LED11 -> unconnected-(U1-PA11/PA9-Pad22)
- U1 pad 23: /LED12 -> unconnected-(U1-PA12/PA10-Pad23)
- U1 pad 24: /SWDIO -> Net-(U1-PA13)
- U1 pad 25: /SWCLK -> Net-(U1-PA14)
Routing:
- net /coil_{+}: track 651.2 -> 0.00 mm, vias 2 -> 0
- net /LED9: track 32.6 -> 6.03 mm, vias 0 -> 2
- net /SWDIO: track 21.9 -> 8.19 mm
- net Net-(U1-PA13): track 0.00 -> 12.6 mm
- net /LED10: track 34.0 -> 21.6 mm
- net /LED4: track 109.0 -> 97.7 mm
- net Net-(U1-PA14): track 0.00 -> 10.7 mm
- net /LED16: track 44.1 -> 33.4 mm
- net GND: track 23.7 -> 13.6 mm, vias 1 -> 5
- net /SWCLK: track 18.7 -> 9.03 mm
- net Net-(R13-Pad2): track 0.00 -> 4.07 mm
- net VDD: track 49.8 -> 53.3 mm
- net /LED17: track 37.2 -> 33.9 mm
- net +BATT: track 23.7 -> 20.5 mm, vias 3 -> 4
- net Net-(D21-A): track 39.7 -> 38.2 mm
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- added copper zone on In6.Cu, net +BATT
- added copper zone on In1.Cu, net GND
- added copper zone on In2.Cu, net GND
- added copper zone on In3.Cu, net GND
- added copper zone on In4.Cu, net GND
- added copper zone on In5.Cu, net GND
- added copper zone on In6.Cu, net GND
- removed copper zone on In2.Cu, net +BATT
Other:
- copper layers 4 -> 8
- board text added: "CJG"
- board text added: "rev1"

Commit message: fuck this lol
Parts:
- removed R11, R12, R13: 0, Resistor_SMD:R_0402_1005Metric
- added C3: 1u, footprints:C_0402_nosilk, F.Cu at (50.0, 44.6)
- added C4: .1u, footprints:C_0402_nosilk, F.Cu at (52.0, 44.6)
- added TP1: TestPoint, footprints:testpoint_better, F.Cu at (60.2, 27.1)
- added TP5: TestPoint, footprints:testpoint_better, F.Cu at (41.5, 25.7)
- added TP6: TestPoint, footprints:testpoint_better, F.Cu at (39.5, 25.7)
- added TP7: TestPoint, footprints:testpoint_better, F.Cu at (53.6, 44.4)
- BT1: footprint footprints:LIR2032 -> footprints:bat_holder
- moved D64 61.9 mm to (52.6, 46.2)
- moved D74 61.9 mm to (52.6, 26.8)
- moved R6 61.9 mm to (54.8, 30.1)
- moved BT1 61.9 mm to (50.0, 36.5), turned to 0 degrees
- moved C1 61.9 mm to (56.0, 38.4)
- moved C2 61.9 mm to (56.0, 35.5)
- moved D1 61.9 mm to (50.0, 24.5)
- moved D10 61.9 mm to (39.1, 31.4)
- moved D11 61.9 mm to (38.6, 32.8)
- moved D12 61.9 mm to (38.2, 34.3)
- moved D13 61.9 mm to (38.0, 35.7)
- moved D14 61.9 mm to (38.0, 37.3)
- moved D15 61.9 mm to (38.2, 38.7)
- moved D16 61.9 mm to (38.6, 40.2)
- moved D17 61.9 mm to (39.1, 41.6)
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Connections:
- TP2 pad 2: Net-(R13-Pad2) -> +BATT
- U1 pad 24: Net-(U1-PA13) -> /SWDIO
- U1 pad 25: Net-(U1-PA14) -> /SWCLK
- U1 pad 6: unconnected-(U1-PF2-Pad6) -> /NRST
Routing:
- net +BATT: track 20.5 -> 36.6 mm, vias 4 -> 2
- net /SWDIO: track 8.19 -> 21.5 mm
- net /SWCLK: track 9.03 -> 21.8 mm
- net Net-(U1-PA13): track 12.6 -> 0.00 mm
- net Net-(U1-PA14): track 10.7 -> 0.00 mm
- net GND: track 13.6 -> 9.14 mm, vias 5 -> 7
- net VDD: track 53.3 -> 57.5 mm
- net Net-(R13-Pad2): track 4.07 -> 0.00 mm
- net /NRST: track 0.00 -> 3.83 mm
- net Net-(D51-K): track 63.3 -> 61.6 mm
- net /LED14: track 30.0 -> 31.1 mm
- net /LED13: track 29.2 -> 30.1 mm
- net Net-(U1-PA0): track 8.21 -> 7.52 mm
- removed copper zone on B.Cu, net +BATT
- removed copper zone on In6.Cu, net +BATT
Other:
- outline, holes or cut-outs redrawn
- board text added: "+"

Commit message: aa
Parts:
- R1, R2, R3, R4, R5: footprint footprints:R_0402_nosilk -> footprints:R_0402_nosilk_square
- moved C2 3.17 mm to (57.0, 38.5), turned to -90 degrees
- moved U2 2.78 mm to (58.2, 38.6)
- moved C1 2.33 mm to (57.7, 40.0)
- moved R9 1.95 mm to (57.1, 41.0)
- moved R10 1.77 mm to (56.8, 42.0)
Routing:
- net VDD: track 57.5 -> 47.4 mm, vias 2 -> 3
- net GND: track 9.14 -> 0.00 mm, vias 7 -> 6
- net /LED4: track 97.8 -> 93.1 mm
- net /LED16: track 33.4 -> 28.7 mm
- net /LED10: track 21.6 -> 17.2 mm
- net +BATT: track 36.6 -> 40.5 mm
- net /LED17: track 33.9 -> 37.0 mm
- net /LED9: track 6.03 -> 7.24 mm
- net /LED12: track 18.6 -> 17.6 mm
- net /LED11: track 16.9 -> 15.9 mm
- net Net-(D21-A): track 38.2 -> 39.1 mm
- removed copper zone on F.Cu, net +BATT
- removed copper zone on F.Cu, net VDD
Other:
- board text added: "rev2"
