File: pcb/watch/watch.kicad_pcb (KiCad board)
At the start: 8 copper layers, 28 x 34.7 mm, 98 parts, among them U1 STM32G031K8Ux, U2 TLV74130PDQNR

Commit message: eee
Parts:
- D10, D12, D13, D14, D15, D16, D17, D18, D19, D2, D20, D22, D23, D24, D25, D26, D27, D28, D29, D3, D30, D32, D33, D34, D35, D36, D37, D38, D39, D4, D40, D42, D43, D44, D45, D46, D47, D48, D49, D5, D50, D6, D7, D8, D9: footprint LED_SMD:LED_0402_1005Metric -> footprints:LED_0402_nosilk
- TP2, TP4: value TestPoint_2Pole -> TestPoint; footprint footprints:tesptoint_tiny -> footprints:testpoint_better_square
- TP3: value TestPoint_2Pole -> TestPoint; footprint footprints:tesptoint_tiny -> footprints:testpoint_better
- moved TP3 30.3 mm to (57.1, 49.3), turned to 90 degrees
- moved R8 12.5 mm to (46.2, 40.3), turned to 90 degrees
- moved R7 10.8 mm to (53.7, 39.9), turned to 90 degrees
- moved R6 6.90 mm to (58.5, 35.9)
- moved TP2 3.48 mm to (60.4, 45.9)
- moved TP4 2.57 mm to (56.7, 23.8)
- moved TP5 2.23 mm to (43.0, 24.0)
- moved TP6 1.40 mm to (39.4, 27.1)
- moved TP1 0.19 mm to (60.4, 27.0)
- moved R10 0.15 mm to (56.6, 42.0), turned to 180 degrees
- moved C3 0.12 mm to (50.0, 44.7)
- moved C4 0.05 mm to (52.0, 44.7)
Connections:
- TP3 pad 1: /SWCLK -> +BATT
Routing:
- net /LED13: track 30.1 -> 1.56 mm, vias 2 -> 0
- net /LED12: track 17.6 -> 1.26 mm
- net Net-(D53-K): track 63.8 -> 72.5 mm, vias 4 -> 5
- net Net-(D55-K): track 61.0 -> 68.4 mm
- net /LED6: track 33.7 -> 26.9 mm
- net /LED11: track 15.9 -> 9.81 mm
- net /LED17: track 37.0 -> 33.3 mm
- net VDD: track 47.4 -> 43.9 mm, vias 3 -> 4
- net /SWCLK: track 21.8 -> 18.6 mm, vias 1 -> 2
- net +BATT: track 40.5 -> 43.4 mm, vias 2 -> 3
- net Net-(D21-A): track 39.1 -> 41.1 mm
- net /SWDIO: track 21.5 -> 19.6 mm, vias 1 -> 2
- net Net-(D51-K): track 61.6 -> 60.4 mm, vias 5 -> 4
- net /LED14: track 31.1 -> 29.9 mm
- net /LED16: track 28.7 -> 29.9 mm
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Other:
- board size 28 x 34.7 mm -> 28 x 34.4 mm
- board text removed: "rev1"

Commit message: e
Parts:
- moved TP6 0.22 mm to (39.3, 27.3)
Changed lines of the file:
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@@
   )
   (footprint "footprints:testpoint_better" (layer "F.Cu")
-    (at 39.4 27.1)
+    (at 39.3 27.3)
     (descr "SMD pad as test Point, diameter 1.0mm")
     (tags "test point SMD pad")
@@
   (segment (start 50.98665 44.20665) (end 50.72 43.94) (width 0.0889) (layer "F.Cu") (net 34))
   (segment (start 47.0778 38.7953) (end 47.0778 37.494904) (width 0.0889) (layer "F.Cu") (net 36))
-  (segment (start 41 26.8) (end 40.7 27.1) (width 0.0889) (layer "F.Cu") (net 36))
   (segment (start 47.0778 37.494904) (end 42.2922 32.709304) (width 0.0889) (layer "F.Cu") (net 36))
+  (segment (start 39.3 27.3) (end 40.5 27.3) (width 0.0889) (layer "F.Cu") (net 36))
+  (segment (start 40.5 27.3) (end 41 26.8) (width 0.0889) (layer "F.Cu") (net 36))
   (segment (start 47.5325 39.25) (end 47.0778 38.7953) (width 0.0889) (layer "F.Cu") (net 36))
   (segment (start 42.2922 32.709304) (end 42.2922 30.7222) (width 0.0889) (layer "F.Cu") (net 36))
   (segment (start 42.2922 30.7222) (end 41.71 30.14) (width 0.0889) (layer "F.Cu") (net 36))
-  (segment (start 40.7 27.1) (end 39.4 27.1) (width 0.0889) (layer "F.Cu") (net 36))
   (via (at 41.71 30.14) (size 0.45) (drill 0.3) (layers "F.Cu" "B.Cu") (net 36))
   (via (at 41 26.8) (size 0.45) (drill 0.3) (layers "F.Cu" "B.Cu") (net 36))

Commit message: rev2 final commit
Parts:
- added H1: MountingHole, footprints:m1.4_hole, F.Cu at (23.4, 45.6)
- added H2: MountingHole, footprints:m1.4_hole, F.Cu at (42.1, 22.6)
- added H3: MountingHole, footprints:m1.4_hole, F.Cu at (23.4, 22.6)
- added H4: MountingHole, footprints:m1.4_hole, F.Cu at (42.1, 45.6)
- added J1: Conn_01x07, footprints:mypinheader, F.Cu at (58.4, 16.0)
- added J2: Conn_01x07, footprints:mypinheader, F.Cu at (58.3, 52.1)
- added J3: Conn_01x07_MountingPin, Connector_JST:JST_GH_SM07B-GHS-TB_1x07-1MP_P1.25mm_Horizontal, F.Cu at (57.8, 34.3)
- added TPM1: TestPoint, footprints:pogo, F.Cu at (69.7, 42.0)
- added TPM2: TestPoint, footprints:pogo, F.Cu at (73.2, 46.9)
- added TPM3: TestPoint, footprints:pogo, F.Cu at (76.5, 24.6)
- added TPM4: TestPoint, footprints:pogo, F.Cu at (72.8, 21.4)
- added TPM5: TestPoint, footprints:pogo, F.Cu at (76.5, 43.5)
- added TPM6: TestPoint, footprints:pogo, F.Cu at (59.1, 21.6)
- added TPM7: TestPoint, footprints:pogo, F.Cu at (55.4, 24.9)
- moved BT1 17.4 mm to (32.8, 34.1)
- moved C2 17.4 mm to (34.8, 42.4)
- moved C3 17.4 mm to (40.5, 37.6)
- moved C4 17.4 mm to (39.8, 36.2)
- moved D28 17.4 mm to (35.8, 45.8)
- moved D29 17.4 mm to (37.2, 45.3)
- moved D30 17.4 mm to (38.6, 44.7)
- moved D31 17.4 mm to (39.8, 43.9)
- moved D35 17.4 mm to (43.6, 39.3)
- moved D42 17.4 mm to (43.6, 29.0)
- moved D46 17.4 mm to (39.8, 24.4)
- moved D47 17.4 mm to (38.6, 23.6)
- moved D48 17.4 mm to (37.2, 23.0)
- moved D49 17.4 mm to (35.8, 22.5)
- moved D52 17.4 mm to (30.2, 24.5)
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- renumbered C3 to C1, C4 to C2, C1 to C3, C2 to C4, TP7 to TP1, TP3 to TP2, TP1 to TP3, TP2 to TP5, TP5 to TP6, TP6 to TP7, U2 to U1, U1 to U2
Routing:
- net /TP_{VDD}: track 0.00 -> 81.4 mm, vias 0 -> 1
- net /TP_{VBAT}: track 0.00 -> 68.7 mm, vias 0 -> 1
- net /TP_{NRST}: track 0.00 -> 66.9 mm, vias 0 -> 1
- net /TP_{SWCLK}: track 0.00 -> 63.6 mm, vias 0 -> 1
- net /TP_{SWDIO}: track 0.00 -> 47.5 mm, vias 0 -> 1
- added copper zone on B.Cu, net /TP_{GND}
- added copper zone on F.Cu, net /TP_{GND}
- added copper zone on In1.Cu, net /TP_{GND}
- added copper zone on In2.Cu, net /TP_{GND}
Other:
- board size 28 x 34.4 mm -> 63.4 x 41.4 mm
- board text added: "CJG rev2"
- board text added: "CLK DIO GND GND VDD VBT RST"
- board text added: "RST VBT VDD GND GND DIO CLK"
- board text added: "pogo"
- board text removed: "+"
