File: pcb/watch/watch.kicad_sch (KiCad schematic)
At the start: 106 parts

Commit message: fuck fuck fuck I made it too small
Parts:
- removed D19 (x25), D49 (x2): LED_Small_Filled, LED_SMD:LED_0402_1005Metric, symbol Device:LED_Small_Filled
- removed R1 (x2), R10, R11, R12, R13, R14, R15, R16, R17, R18, R19, R2 (x2), R20, R21, R22, R23, R24, R3 (x2), R4 (x2), R5 (x2), R6 (x2), R7 (x3), R9: R_Small_US, Resistor_SMD:R_0402_1005Metric, symbol Device:R_Small_US
- added D19, D49, D50, D51, D52, D53, D54, D55, D56, D57, D58, D59, D60, D61, D62, D63, D64, D65, D66, D67, D68, D69, D70, D71, D72, D73, D74: LED_Small_Filled, LED_SMD:LED_0402_1005Metric, symbol Device:LED_Small_Filled
- added R1, R2, R3, R4, R5, R6, R7: R_Small_US, Resistor_SMD:R_0402_1005Metric, symbol Device:R_Small_US
- added U1: STM32G031K8Ux, Package_DFN_QFN:UFQFPN-32-1EP_5x5mm_P0.5mm_EP3.5x3.5mm, symbol MCU_ST_STM32G0:STM32G031K8Ux
- D1, D11, D21, D31, D41: footprint LED_SMD:LED_0402_1005Metric -> footprints:LED_0402_1005Metric
Connections:
- net GND: now also U1.33 (VSS), U1.5 (VSS)
- net at R8.2: now also D55.1 (K), D56.2 (A), D61.1 (K), D62.2 (A), D67.1 (K), D68.2 (A), D73.1 (K), D74.2 (A)
- removed net GPIO_{1}: D1.1 (K), D10.1 (K), D13.1 (K), D16.1 (K), D2.1 (K), D3.1 (K)
- removed net GPIO_{2}: D11.1 (K), D14.1 (K), D17.1 (K), D20.1 (K), D4.1 (K), D5.1 (K), D6.1 (K)
- net GPIO_{35} renamed LED13
- net LED13: now also U1.18 (PA8)
- removed net GPIO_{3}: D12.1 (K), D15.1 (K), D18.1 (K), D21.1 (K), D7.1 (K), D8.1 (K), D9.1 (K)
- removed net GPIO_{4}: D22.1 (K), D25.1 (K), D28.1 (K), D31.1 (K), D34.1 (K), D37.1 (K), D40.1 (K)
- removed net GPIO_{5}: D23.1 (K), D26.1 (K), D29.1 (K), D32.1 (K), D35.1 (K), D38.1 (K), D41.1 (K)
- removed net GPIO_{6}: D24.1 (K), D27.1 (K), D30.1 (K), D33.1 (K), D36.1 (K), D39.1 (K), D42.1 (K)
- net GPIO_{7}: no longer names the net of D44.1 (K), D46.1 (K), D48.1 (K)
- net GPIO_{7}: now also D41.2 (A), D42.1 (K), D43.2 (A), D45.2 (A), D47.2 (A), D49.2 (A), D50.1 (K), R5.1; no longer D43.1 (K), D45.1 (K), D47.1 (K)
- new net: D53.1 (K), D54.2 (A), D59.1 (K), D60.2 (A), D65.1 (K), D66.2 (A), D71.1 (K), D72.2 (A), R7.2
- new net: D1.2 (A), D10.1 (K), D2.1 (K), D3.2 (A), D4.1 (K), D5.2 (A), D6.1 (K), D7.2 (A), D8.1 (K), D9.2 (A), R1.1
- new net: D11.2 (A), D12.1 (K), D13.2 (A), D14.1 (K), D15.2 (A), D16.1 (K), D17.2 (A), D18.1 (K), D19.2 (A), D20.1 (K), R2.1
- new net: D31.2 (A), D32.1 (K), D33.2 (A), D34.1 (K), D35.2 (A), D36.1 (K), D37.2 (A), D38.1 (K), D39.2 (A), D40.1 (K), R4.1
- new net: D51.1 (K), D52.2 (A), D57.1 (K), D58.2 (A), D63.1 (K), D64.2 (A), D69.1 (K), D70.2 (A), R6.2
- new net: D21.2 (A), D22.1 (K), D23.2 (A), D24.1 (K), D25.2 (A), D26.1 (K), D27.2 (A), D28.1 (K), D29.2 (A), D30.1 (K), R3.1
- new net LED1: D1.1 (K), D11.1 (K), D12.2 (A), D2.2 (A), D21.1 (K), D22.2 (A), D31.1 (K), D32.2 (A), D41.1 (K), D42.2 (A), U1.1 (PB9)
- new net LED10: R5.2, U1.15 (PB0)
- new net LED11: R6.1, U1.16 (PB1)
- new net LED12: R7.1, U1.17 (PB2)
- new net LED14: D51.2 (A), D52.1 (K), D53.2 (A), D54.1 (K), D55.2 (A), D56.1 (K), U1.22 (PA11/PA9)
- new net LED15: D57.2 (A), D58.1 (K), D59.2 (A), D60.1 (K), D61.2 (A), D62.1 (K), U1.3 (PC15)
- new net LED16: D63.2 (A), D64.1 (K), D65.2 (A), D66.1 (K), D67.2 (A), D68.1 (K), U1.9 (PA2)
- new net LED17: D69.2 (A), D70.1 (K), D71.2 (A), D72.1 (K), D73.2 (A), D74.1 (K), U1.19 (PA9/NC)
- new net LED2: D13.1 (K), D14.2 (A), D23.1 (K), D24.2 (A), D3.1 (K), D33.1 (K), D34.2 (A), D4.2 (A), D43.1 (K), D44.2 (A), U1.26 (PA15)
- new net LED3: D15.1 (K), D16.2 (A), D25.1 (K), D26.2 (A), D35.1 (K), D36.2 (A), D45.1 (K), D46.2 (A), D5.1 (K), D6.2 (A), U1.6 (PF2)
- new net LED4: D17.1 (K), D18.2 (A), D27.1 (K), D28.2 (A), D37.1 (K), D38.2 (A), D47.1 (K), D48.2 (A), D7.1 (K), D8.2 (A), U1.10 (PA3)
- new net LED5: D10.2 (A), D19.1 (K), D20.2 (A), D29.1 (K), D30.2 (A), D39.1 (K), D40.2 (A), D49.1 (K), D50.2 (A), D9.1 (K), U1.20 (PC6)
- new net LED6: R1.2, U1.21 (PA10/NC)
- new net LED7: R2.2, U1.25 (PA14)
- new net LED8: R3.2, U1.2 (PC14)
- new net LED9: R4.2, U1.8 (PA1)
- new net VDD: U1.4 (VDD)
Other:
- note added: "Minutes+Hours"
- note removed: "Hours"
- note removed: "Minutes"

Commit message: eee
Parts:
- added BT1: LIR2032, footprints:LIR2032, symbol Device:Battery_Cell
- added C1, C2: 1u, footprints:C_0402_nosilk, symbol Device:C_Small
- added L1: ~, symbol Device:L
- added R10, R9: 169k, footprints:LED_0402_nosilk, symbol Device:R_Small_US
- added TP1, TP2, TP3, TP4: TestPoint_2Pole, footprints:tesptoint_tiny, symbol Connector:TestPoint_2Pole
- added U2: TLV74130PDQNR, footprints:Texas_X2SON_nosilk, symbol symbol_library:TLV74130PDQNR
- D52, D53, D54, D55, D56, D57, D58, D59, D60, D61, D62, D63, D64, D65, D66, D67, D68, D69, D70, D71, D72, D73, D74: footprint LED_SMD:LED_0402_1005Metric -> footprints:LED_0402_nosilk
- R1, R2, R3, R4, R5, R6, R7, R8: footprint Resistor_SMD:R_0402_1005Metric -> footprints:R_0402_nosilk
- U1: footprint Package_DFN_QFN:UFQFPN-32-1EP_5x5mm_P0.5mm_EP3.5x3.5mm -> footprints:UFQFPN-32-nosilk
Connections:
- net GND: now also U1.3 (PC15), BT1.2 (-), C1.2, C2.2, R10.2, TP2.1, TP4.1, U2.2 (CASE), U2.5 (GND)
- net LED1: now also U1.31 (PB7); no longer U1.1 (PB9)
- net LED10: now also U1.11 (PA4); no longer U1.15 (PB0)
- net LED14: now also U1.23 (PA12/PA10); no longer U1.22 (PA11/PA9)
- net LED15: now also U1.1 (PB9); no longer U1.3 (PC15)
- net LED3: now also U1.2 (PC14); no longer U1.6 (PF2)
- net LED5: now also U1.21 (PA10/NC); no longer U1.20 (PC6)
- net LED6: now also U1.20 (PC6); no longer U1.21 (PA10/NC)
- net LED7: now also U1.27 (PB3); no longer U1.25 (PA14)
- net LED8: now also U1.32 (PB8); no longer U1.2 (PC14)
- net VDD: now also C2.1, TP4.2, U2.1 (V_{out})
- net SWDIO: now reaches U1.24 (PA13)
- net SWDIO: now also TP3.2
- net at U1.7 (PA0): now also R10.1, R9.2
- new net +BATT: BT1.1 (+), C1.1, R9.1, TP2.2, U2.3 (EN), U2.4 (V_{in})
- new net SWCLK: TP3.1, U1.25 (PA14)
- new net coil_{+}: L1.1, TP1.1, TP1.2
Other:
- note added: "Vdd = 3.0v"
- note added: "max: 4.2v min: 3.0v"
- note added: "we just route it correctly in the pcd"

Commit message: eeeee
Connections:
- net GND: no longer U1.3 (PC15)
- net LED1: now also U1.32 (PB8); no longer U1.31 (PB7)
- net LED11: now also U1.22 (PA11/PA9); no longer U1.16 (PB1)
- net LED12: now also U1.23 (PA12/PA10); no longer U1.17 (PB2)
- net LED13: now also U1.27 (PB3); no longer U1.18 (PA8)
- net LED14: now also U1.26 (PA15); no longer U1.23 (PA12/PA10)
- net LED15: now also U1.2 (PC14); no longer U1.1 (PB9)
- net LED17: now also U1.21 (PA10/NC); no longer U1.19 (PA9/NC)
- net LED2: now also U1.29 (PB5); no longer U1.26 (PA15)
- net LED3: now also U1.3 (PC15); no longer U1.2 (PC14)
- net LED5: now also U1.31 (PB7); no longer U1.21 (PA10/NC)
- net LED6: now also U1.30 (PB6); no longer U1.20 (PC6)
- net LED7: now also U1.28 (PB4); no longer U1.27 (PB3)
- net LED8: now also U1.1 (PB9); no longer U1.32 (PB8)
Changed lines of the file:
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@@
   (junction (at 269.24 33.02) (diameter 0) (color 0 0 0 0)
   )
-  (junction (at 148.59 77.47) (diameter 0) (color 0 0 0 0)
-  )
   (junction (at 86.36 29.21) (diameter 0) (color 0 0 0 0)
   )
@@
     (stroke (width 0) (type default))
   )
-  (wire (pts (xy 124.46 77.47) (xy 148.59 77.47))
-    (stroke (width 0) (type default))
-  )
   (wire (pts (xy 218.44 33.02) (xy 229.87 33.02))
     (stroke (width 0) (type default))
@@
     (stroke (width 0) (type default))
   )
-  (wire (pts (xy 124.46 40.64) (xy 124.46 77.47))
-    (stroke (width 0) (type default))
-  )
   (wire (pts (xy 45.72 63.5) (xy 45.72 69.85))
     (stroke (width 0) (type default))
@@
     (stroke (width 0) (type default))
   )
-  (wire (pts (xy 148.59 78.74) (xy 148.59 77.47))
-    (stroke (width 0) (type default))
-  )
   (wire (pts (xy 92.71 33.02) (xy 92.71 36.83))
     (stroke (width 0) (type default))
@@
     (stroke (width 0) (type default))
   )
-  (wire (pts (xy 133.35 40.64) (xy 124.46 40.64))
-    (stroke (width 0) (type default))
-  )
   (wire (pts (xy 110.49 33.02) (xy 110.49 36.83))
     (stroke (width 0) (type default))
@@
     (stroke (width 0) (type default))
   )
-  (wire (pts (xy 148.59 77.47) (xy 148.59 76.2))
+  (wire (pts (xy 148.59 76.2) (xy 148.59 78.74))
     (stroke (width 0) (type default))
   )
@@
     (effects (font (size 4 4)) (justify left bottom))
   )
-  (label "LED7" (at 133.35 53.34 180) (fields_autoplaced)
-    (effects (font (size 1.27 1.27)) (justify right bottom))
-  )
-  (label "LED6" (at 133.35 35.56 180) (fields_autoplaced)
-    (effects (font (size 1.27 1.27)) (justify right bottom))
-  )
-  (label "LED8" (at 133.35 66.04 180) (fields_autoplaced)
+  (label "LED7" (at 133.35 55.88 180) (fields_autoplaced)
+    (effects (font (size 1.27 1.27)) (justify right bottom))
+  )
+  (label "LED6" (at 133.35 60.96 180) (fields_autoplaced)
+    (effects (font (size 1.27 1.27)) (justify right bottom))
+  )
+  (label "LED8" (at 133.35 68.58 180) (fields_autoplaced)
     (effects (font (size 1.27 1.27)) (justify right bottom))
   )
@@
     (effects (font (size 1.27 1.27)) (justify left bottom))
   )
-  (label "LED13" (at 161.29 50.8 0) (fields_autoplaced)
-    (effects (font (size 1.27 1.27)) (justify left bottom))
+  (label "LED13" (at 133.35 53.34 180) (fields_autoplaced)
+    (effects (font (size 1.27 1.27)) (justify right bottom))
   )
   (label "LED5" (at 26.67 76.2 180) (fields_autoplaced)
@@
     (effects (font (size 1.27 1.27)) (justify right bottom))
   )
-  (label "LED17" (at 161.29 53.34 0) (fields_autoplaced)
+  (label "LED17" (at 161.29 55.88 0) (fields_autoplaced)
     (effects (font (size 1.27 1.27)) (justify left bottom))
   )
@@
     (effects (font (size 1.27 1.27)) (justify left bottom))
   )
-  (label "LED15" (at 133.35 68.58 180) (fields_autoplaced)
+  (label "LED15" (at 133.35 38.1 180) (fields_autoplaced)
     (effects (font (size 1.27 1.27)) (justify right bottom))
   )
@@
     (effects (font (size 1.27 1.27)) (justify left bottom))
   )
-  (label "LED2" (at 161.29 68.58 0) (fields_autoplaced)
-    (effects (font (size 1.27 1.27)) (justify left bottom))
+  (label "LED2" (at 133.35 58.42 180) (fields_autoplaced)
+    (effects (font (size 1.27 1.27)) (justify right bottom))
   )
   (label "LED9" (at 161.29 33.02 0) (fields_autoplaced)
     (effects (font (size 1.27 1.27)) (justify left bottom))
   )
-  (label "LED5" (at 161.29 55.88 0) (fields_autoplaced)
-    (effects (font (size 1.27 1.27)) (justify left bottom))
+  (label "LED5" (at 133.35 63.5 180) (fields_autoplaced)
+    (effects (font (size 1.27 1.27)) (justify right bottom))
   )
   (label "SWDIO" (at 161.29 63.5 0) (fields_autoplaced)
@@
     (effects (font (size 1.27 1.27)) (justify left bottom))
   )
-  (label "LED12" (at 133.35 50.8 180) (fields_autoplaced)
-    (effects (font (size 1.27 1.27)) (justify right bottom))
-  )
-  (label "LED1" (at 133.35 63.5 180) (fields_autoplaced)
+  (label "LED12" (at 161.29 60.96 0) (fields_autoplaced)
+    (effects (font (size 1.27 1.27)) (justify left bottom))
+  )
+  (label "LED1" (at 133.35 66.04 180) (fields_autoplaced)
     (effects (font (size 1.27 1.27)) (justify right bottom))
   )
@@
     (effects (font (size 1.27 1.27)) (justify right bottom))
   )
-  (label "LED3" (at 133.35 38.1 180) (fields_autoplaced)
+  (label "LED3" (at 133.35 40.64 180) (fields_autoplaced)
     (effects (font (size 1.27 1.27)) (justify right bottom))
   )
@@
     (effects (font (size 1.27 1.27)) (justify left bottom))
   )
-  (label "LED14" (at 161.29 60.96 0) (fields_autoplaced)
+  (label "LED14" (at 161.29 68.58 0) (fields_autoplaced)
     (effects (font (size 1.27 1.27)) (justify left bottom))
   )
@@
     (effects (font (size 1.27 1.27)) (justify left bottom))
   )
-  (label "LED11" (at 133.35 48.26 180) (fields_autoplaced)
-    (effects (font (size 1.27 1.27)) (justify right bottom))
+  (label "LED11" (at 161.29 58.42 0) (fields_autoplaced)
+    (effects (font (size 1.27 1.27)) (justify left bottom))
   )
   (label "LED3" (at 26.67 55.88 180) (fields_autoplaced)

Commit message: e
Other:
- note added: "LCSC: C965796 for white LEDS. V_f = 2.6-2.8 LCSC: C965790 for red LEDS. V_f = 1.9-2.1"
Changed lines of the file:
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@@
     (effects (font (size 4 4)) (justify left bottom))
+  )
+  (text "LCSC:  C965796 for white LEDS. V_f = 2.6-2.8\nLCSC:  C965790 for red   LEDS. V_f = 1.9-2.1"
+    (at 44.45 92.71 0)
+    (effects (font (size 1.27 1.27)) (justify left bottom))
   )
   (label "LED7" (at 133.35 55.88 180) (fields_autoplaced)

Commit message: rev1 lol
Parts:
- removed L1: ~, symbol Device:L
- removed TP1: TestPoint_2Pole, footprints:tesptoint_tiny, symbol Connector:TestPoint_2Pole
- added R11, R12, R13: 0, Resistor_SMD:R_0402_1005Metric, symbol Device:R_Small_US
Connections:
- net +BATT: now also R13.1; no longer TP2.2
- net LED11: now also U1.13 (PA6); no longer U1.22 (PA11/PA9)
- net LED12: now also U1.14 (PA7); no longer U1.23 (PA12/PA10)
- net LED17: now also U1.12 (PA5); no longer U1.21 (PA10/NC)
- net SWCLK: now also R11.2; no longer U1.25 (PA14)
- net SWDIO: now also R12.2; no longer U1.24 (PA13)
- new net: R13.2, TP2.2
- new net: R11.1, U1.25 (PA14)
- new net: R12.1, U1.24 (PA13)
Other:
- note removed: "we just route it correctly in the pcd"
- moved on the sheet: TP2, TP3

Commit message: fuck this lol
Parts:
- removed R11, R12, R13: 0, Resistor_SMD:R_0402_1005Metric, symbol Device:R_Small_US
- added C3: 1u, footprints:C_0402_nosilk, symbol Device:C_Small
- added C4: .1u, footprints:C_0402_nosilk, symbol Device:C_Small
- added TP1, TP5, TP6, TP7: TestPoint, footprints:testpoint_better, symbol Connector:TestPoint
- BT1: footprint footprints:LIR2032 -> footprints:bat_holder
Connections:
- net +BATT: now also TP2.2
- net GND: now also C3.2, C4.2
- net SWCLK: now also U1.25 (PA14), TP6.1
- net SWDIO: now also U1.24 (PA13), TP5.1
- net VDD: now also C3.1, TP1.1
- net NRST: now reaches U1.6 (PF2)
- net NRST: now also C4.1, TP7.1
Other:
- moved on the sheet: D51, D52, D53, D54, D55, D56, D57, D58, D59, D60, D61, D62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

Commit message: aa
Parts:
- R1, R2, R3, R4, R5: footprint footprints:R_0402_nosilk -> footprints:R_0402_nosilk_square
Changed lines of the file:
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@@
       (effects (font (size 1.27 1.27)) (justify left) hide)
     )
-    (property "Footprint" "footprints:R_0402_nosilk" (at 45.72 30.48 0)
+    (property "Footprint" "footprints:R_0402_nosilk_square" (at 45.72 30.48 0)
       (effects (font (size 1.27 1.27)) hide)
     )
@@
       (effects (font (size 1.27 1.27)) (justify left) hide)
     )
-    (property "Footprint" "footprints:R_0402_nosilk" (at 39.37 30.48 0)
+    (property "Footprint" "footprints:R_0402_nosilk_square" (at 39.37 30.48 0)
       (effects (font (size 1.27 1.27)) hide)
     )
@@
       (effects (font (size 1.27 1.27)) (justify left) hide)
     )
-    (property "Footprint" "footprints:R_0402_nosilk" (at 52.07 30.48 0)
+    (property "Footprint" "footprints:R_0402_nosilk_square" (at 52.07 30.48 0)
       (effects (font (size 1.27 1.27)) hide)
     )
@@
       (effects (font (size 1.27 1.27)) (justify left) hide)
     )
-    (property "Footprint" "footprints:R_0402_nosilk" (at 58.42 30.48 0)
+    (property "Footprint" "footprints:R_0402_nosilk_square" (at 58.42 30.48 0)
       (effects (font (size 1.27 1.27)) hide)
     )
@@
       (effects (font (size 1.27 1.27)) (justify left) hide)
     )
-    (property "Footprint" "footprints:R_0402_nosilk" (at 33.02 30.48 0)
-      (effects (font (size 1.27 1.27)) hide)
-    )
+    (property "Footprint" "footprints:R_0402_nosilk_square" (at 33.02 30.48 0)
+      (effects (font (size 1.27 1.27)) hide)
+    )

Commit message: eee
Parts:
- removed TP2, TP3, TP4: TestPoint_2Pole, footprints:tesptoint_tiny, symbol Connector:TestPoint_2Pole
- added TP2, TP4: TestPoint, footprints:testpoint_better_square, symbol Connector:TestPoint
- added TP3: TestPoint, footprints:testpoint_better, symbol Connector:TestPoint
- D10, D12, D13, D14, D15, D16, D17, D18, D19, D2, D20, D22, D23, D24, D25, D26, D27, D28, D29, D3, D30, D32, D33, D34, D35, D36, D37, D38, D39, D4, D40, D42, D43, D44, D45, D46, D47, D48, D49, D5, D50, D6, D7, D8, D9: footprint LED_SMD:LED_0402_1005Metric -> footprints:LED_0402_nosilk
Connections:
- net +BATT: now also TP3.1
- net GND: now also TP2.1, TP4.1
Other:
- moved on the sheet: TP5, TP6
