File: pcb/watch/watch.kicad_sch (KiCad schematic)
At the start: 98 parts, among them U1 STM32G031K8Ux, U2 TLV74130PDQNR

Commit message: rev2 final commit
Parts:
- added H1, H2, H3, H4: MountingHole, footprints:m1.4_hole, symbol Mechanical:MountingHole
- added J1, J2: Conn_01x07, footprints:mypinheader, symbol Connector_Generic:Conn_01x07
- added J3: Conn_01x07_MountingPin, Connector_JST:JST_GH_SM07B-GHS-TB_1x07-1MP_P1.25mm_Horizontal, symbol Connector_Generic_MountingPin:Conn_01x07_MountingPin
- added TPM1, TPM2, TPM3, TPM4, TPM5, TPM6, TPM7: TestPoint, footprints:pogo, symbol Connector:TestPoint
- renumbered C3 to C1, C4 to C2, C1 to C3, C2 to C4, TP7 to TP1, TP3 to TP2, TP1 to TP3, TP2 to TP5, TP5 to TP6, TP6 to TP7, U2 to U1, U1 to U2
Connections:
- new net TP_{GND}: J1.3 (Pin_3), J1.4 (Pin_4), J2.3 (Pin_3), J2.4 (Pin_4), J3.3 (Pin_3), J3.4 (Pin_4), J3.MP (MountPin), TPM4.1, TPM5.1
- new net TP_{NRST}: J1.7 (Pin_7), J2.7 (Pin_7), J3.7 (Pin_7), TPM1.1
- new net TP_{SWCLK}: J1.1 (Pin_1), J2.1 (Pin_1), J3.1 (Pin_1), TPM7.1
- new net TP_{SWDIO}: J1.2 (Pin_2), J2.2 (Pin_2), J3.2 (Pin_2), TPM6.1
- new net TP_{VBAT}: J1.6 (Pin_6), J2.6 (Pin_6), J3.6 (Pin_6), TPM2.1
- new net TP_{VDD}: J1.5 (Pin_5), J2.5 (Pin_5), J3.5 (Pin_5), TPM3.1
